Commit message: xacro URDF improvements

File: urdf/spotmicroai.urdf.xacro (robot description, xacro)
@@ -9,13 +9,4 @@
   <material name="grey">
     <color rgba="0.6 0.6 0.6 1"/>
-  </material>
-  <material name="blue">
-    <color rgba="0 0 0.8 1"/>
-  </material>
-  <material name="green">
-    <color rgba="0 0.9 0 1"/>
-  </material>
-  <material name="red">
-    <color rgba="0.9 0 0 1"/>
   </material>
   <!-- Params -->
@@ -61,13 +52,47 @@
   </xacro:macro>
   <xacro:macro name="gen_toe" params="name">
-     <link name="${name}">
-    <visual>
-      <geometry>
-        <cylinder length="0.020" radius="0.014"/>
-      </geometry>
-      <origin rpy="1.5708 0 0" xyz="0 0 0"/>
-      <material name="grey"/>
-    </visual>
-  </link>
+    <link name="${name}">
+      <visual>
+        <geometry>
+          <cylinder length="0.020" radius="0.014"/>
+        </geometry>
+        <origin rpy="1.5708 0 0" xyz="0 0 0"/>
+        <material name="grey"/>
+      </visual>
+    </link>
+  </xacro:macro>
+  <xacro:macro name="gen_foot_joint" params="pos">
+    <joint name="${pos}_foot" type="revolute">
+      <parent link="${pos}_leg_link"/>
+      <child link="${pos}_foot_link"/>
+      <axis xyz="0 1 0"/>
+      <origin xyz="-0.01 0 -0.120"/>
+      <limit effort="1000.0" lower="-0.1" upper="2.59" velocity="0.5"/>
+    </joint>
+  </xacro:macro>
+  <xacro:macro name="gen_toe_joint" params="pos">
+    <joint name="${pos}_toe" type="fixed">
+      <parent link="${pos}_foot_link"/>
+      <child link="${pos}_toe_link"/>
+      <origin xyz="0 0 -0.155"/>
+    </joint>
+  </xacro:macro>
+  <xacro:macro name="gen_leg_joint" params="pos shift">
+    <joint name="${pos}_leg" type="revolute">
+      <parent link="${pos}_shoulder_link"/>
+      <child link="${pos}_leg_link"/>
+      <axis xyz="0 1 0"/>
+      <origin xyz="0 ${shift} 0"/>
+      <limit effort="1000.0" lower="-2.666" upper="1.548" velocity="0.5"/>
+    </joint>
+  </xacro:macro>
+  <xacro:macro name="gen_shoulder_joint" params="pos shiftx shifty">
+ <joint name="${pos}_shoulder" type="revolute">
+    <parent link="base_link"/>
+    <child link="${pos}_shoulder_link"/>
+    <axis xyz="1 0 0"/>
+    <origin xyz="${shiftx} ${shifty} 0"/>
+    <limit effort="1000.0" lower="-0.548" upper="0.548" velocity="0.5"/>
+  </joint>
   </xacro:macro>
   <!-- Body -->
@@ -128,112 +153,23 @@
     <child link="front_link"/>
   </joint>
-  <!-- ShoulderJoints -->
-  <!-- Front left -->
-  <joint name="base_front_left" type="revolute">
-    <parent link="base_link"/>
-    <child link="front_left_shoulder_link"/>
-    <axis xyz="1 0 0"/>
-    <origin xyz="-0.093 -0.036 0"/>
-    <limit effort="1000.0" lower="-0.548" upper="0.548" velocity="0.5"/>
-  </joint>
-  <joint name="front_left_leg" type="revolute">
-    <parent link="front_left_shoulder_link"/>
-    <child link="front_left_leg_link"/>
-    <axis xyz="0 1 0"/>
-    <origin xyz="0 -0.042 0"/>
-    <limit effort="1000.0" lower="-2.666" upper="1.548" velocity="0.5"/>
-  </joint>
-  <joint name="front_left_foot" type="revolute">
-    <parent link="front_left_leg_link"/>
-    <child link="front_left_foot_link"/>
-    <axis xyz="0 1 0"/>
-    <origin xyz="-0.01 0 -0.120"/>
-    <limit effort="1000.0" lower="-0.1" upper="2.59" velocity="0.5"/>
-  </joint>
-  <joint name="front_left_toe" type="fixed">
-    <parent link="front_left_foot_link"/>
-    <child link="front_left_toe_link"/>
-    <origin xyz="0 0 -0.155"/>
-  </joint>
-  <!-- Front right -->
-  <joint name="base_front_right" type="revolute">
-    <parent link="base_link"/>
-    <child link="front_right_shoulder_link"/>
-    <axis xyz="1 0 0"/>
-    <origin xyz="-0.093 0.036 0"/>
-    <limit effort="1000.0" lower="-0.548" upper="0.548" velocity="0.5"/>
-  </joint>
-  <joint name="front_right_leg" type="revolute">
-    <parent link="front_right_shoulder_link"/>
-    <child link="front_right_leg_link"/>
-    <axis xyz="0 1 0"/>
-    <origin xyz="0 0.042 0"/>
-    <limit effort="1000.0" lower="-2.666" upper="1.548" velocity="0.5"/>
-  </joint>
-  <joint name="front_right_foot" type="revolute">
-    <parent link="front_right_leg_link"/>
-    <child link="front_right_foot_link"/>
-    <axis xyz="0 1 0"/>
-    <origin xyz="-0.01 0 -0.120"/>
-    <limit effort="1000.0" lower="-0.1" upper="2.59" velocity="0.5"/>
-  </joint>
-  <joint name="front_right_toe" type="fixed">
-    <parent link="front_right_foot_link"/>
-    <child link="front_right_toe_link"/>
-    <origin xyz="0 0 -0.155"/>
-  </joint>
-  <!-- rear left -->
-  <joint name="base_rear_left" type="revolute">
-    <parent link="base_link"/>
-    <child link="rear_left_shoulder_link"/>
-    <axis xyz="1 0 0"/>
-    <origin xyz="0.093 -0.036 0"/>
-    <limit effort="1000.0" lower="-0.548" upper="0.548" velocity="0.5"/>
-  </joint>
-  <joint name="rear_left_leg" type="revolute">
-    <parent link="rear_left_shoulder_link"/>
-    <child link="rear_left_leg_link"/>
-    <axis xyz="0 1 0"/>
-    <origin xyz="0 -0.042 0"/>
-    <limit effort="1000.0" lower="-2.666" upper="1.548" velocity="0.5"/>
-  </joint>
-  <joint name="rear_left_foot" type="revolute">
-    <parent link="rear_left_leg_link"/>
-    <child link="rear_left_foot_link"/>
-    <axis xyz="0 1 0"/>
-    <origin xyz="-0.01 0 -0.120"/>
-    <limit effort="1000.0" lower="-0.1" upper="2.59" velocity="0.5"/>
-  </joint>
-  <joint name="rear_left_toe" type="fixed">
-    <parent link="rear_left_foot_link"/>
-    <child link="rear_left_toe_link"/>
-    <origin xyz="0 0 -0.155"/>
-  </joint>
-  <!-- rear right -->
-  <joint name="base_rear_right" type="revolute">
-    <parent link="base_link"/>
-    <child link="rear_right_shoulder_link"/>
-    <axis xyz="1 0 0"/>
-    <origin xyz="0.093 0.036 0"/>
-    <limit effort="1000.0" lower="-0.548" upper="0.548" velocity="0.5"/>
-  </joint>
-  <joint name="rear_right_leg" type="revolute">
-    <parent link="rear_right_shoulder_link"/>
-    <child link="rear_right_leg_link"/>
-    <axis xyz="0 1 0"/>
-    <origin xyz="0 0.042 0"/>
-    <limit effort="1000.0" lower="-2.666" upper="1.548" velocity="0.5"/>
-  </joint>
-  <joint name="rear_right_foot" type="revolute">
-    <parent link="rear_right_leg_link"/>
-    <child link="rear_right_foot_link"/>
-    <axis xyz="0 1 0"/>
-    <origin xyz="-0.01 0 -0.120"/>
-    <limit effort="1000.0" lower="-0.1" upper="2.59" velocity="0.5"/>
-  </joint>
-  <joint name="rear_right_toe" type="fixed">
-    <parent link="rear_right_foot_link"/>
-    <child link="rear_right_toe_link"/>
-    <origin xyz="0 0 -0.155"/>
-  </joint>
+  <!-- Shoulder Joints -->
+  <xacro:gen_shoulder_joint pos="front_left" shiftx="-0.093" shifty="-0.036"/>
+  <xacro:gen_shoulder_joint pos="front_right" shiftx="-0.093" shifty="0.036"/>
+  <xacro:gen_shoulder_joint pos="rear_left" shiftx="0.093" shifty="-0.036"/>
+  <xacro:gen_shoulder_joint pos="rear_right" shiftx="0.093" shifty="0.036"/>
+  <!-- Leg Joints -->
+  <xacro:gen_leg_joint pos="front_left" shift="-0.042"/>
+  <xacro:gen_leg_joint pos="front_right" shift="0.042"/>
+  <xacro:gen_leg_joint pos="rear_left" shift="-0.042"/>
+  <xacro:gen_leg_joint pos="rear_right" shift="0.042"/>
+  <!-- Foot Joints -->
+  <xacro:gen_foot_joint pos="front_left"/>
+  <xacro:gen_foot_joint pos="front_right"/>
+  <xacro:gen_foot_joint pos="rear_left"/>
+  <xacro:gen_foot_joint pos="rear_right"/>
+  <!-- Toe Joints -->
+  <xacro:gen_toe_joint pos="front_left"/>
+  <xacro:gen_toe_joint pos="front_right"/>
+  <xacro:gen_toe_joint pos="rear_left"/>
+  <xacro:gen_toe_joint pos="rear_right"/>
 </robot>

Commit message: further xacro improvements. < 200lines now

File: urdf/spotmicroai.urdf.xacro (robot description, xacro)
@@ -18,4 +18,5 @@
   <xacro:property name="shoulder_length" value="0.044" />
   <xacro:property name="shoulder_width" value="0.038" />
+  <!-- Macros -->
   <xacro:macro name="gen_shoulder" params="name">
     <link name="${name}">
@@ -88,13 +89,23 @@
   </xacro:macro>
   <xacro:macro name="gen_shoulder_joint" params="pos shiftx shifty">
- <joint name="${pos}_shoulder" type="revolute">
-    <parent link="base_link"/>
-    <child link="${pos}_shoulder_link"/>
-    <axis xyz="1 0 0"/>
-    <origin xyz="${shiftx} ${shifty} 0"/>
-    <limit effort="1000.0" lower="-0.548" upper="0.548" velocity="0.5"/>
-  </joint>
+    <joint name="${pos}_shoulder" type="revolute">
+      <parent link="base_link"/>
+      <child link="${pos}_shoulder_link"/>
+      <axis xyz="1 0 0"/>
+      <origin xyz="${shiftx} ${shifty} 0"/>
+      <limit effort="1000.0" lower="-0.548" upper="0.548" velocity="0.5"/>
+    </joint>
   </xacro:macro>
-  <!-- Body -->
+  <xacro:macro name="gen_full_leg_joint" params="pos shiftx shifty shift">
+    <xacro:gen_shoulder name="${pos}_shoulder_link"/>
+    <xacro:gen_leg name="${pos}_leg_link"/>
+    <xacro:gen_foot name="${pos}_foot_link"/>
+    <xacro:gen_toe name="${pos}_toe_link"/>
+    <xacro:gen_shoulder_joint pos="${pos}" shiftx="${shiftx}" shifty="${shifty}"/>
+    <xacro:gen_leg_joint pos="${pos}" shift="${shift}"/>
+    <xacro:gen_foot_joint pos="${pos}"/>
+    <xacro:gen_toe_joint pos="${pos}"/>
+  </xacro:macro>
+  <!-- Robot Body -->
   <link name="base_link">
     <visual>
@@ -115,4 +126,8 @@
     </visual>
   </link>
+  <joint name="base_rear" type="fixed">
+    <parent link="base_link"/>
+    <child link="rear_link"/>
+  </joint>
   <link name="front_link">
     <visual>
@@ -124,52 +139,12 @@
     </visual>
   </link>
-  <!-- Shoulder -->
-  <xacro:gen_shoulder name="front_left_shoulder_link"/>
-  <xacro:gen_shoulder name="front_right_shoulder_link"/>
-  <xacro:gen_shoulder name="rear_left_shoulder_link"/>
-  <xacro:gen_shoulder name="rear_right_shoulder_link"/>
-  <!-- Legs -->
-  <xacro:gen_leg name="front_left_leg_link"/>
-  <xacro:gen_leg name="front_right_leg_link"/>
-  <xacro:gen_leg name="rear_left_leg_link"/>
-  <xacro:gen_leg name="rear_right_leg_link"/>
-  <!-- Feet -->
-  <xacro:gen_foot name="front_left_foot_link"/>
-  <xacro:gen_foot name="front_right_foot_link"/>
-  <xacro:gen_foot name="rear_left_foot_link"/>
-  <xacro:gen_foot name="rear_right_foot_link"/>
-  <!-- Toes -->
-  <xacro:gen_toe name="front_left_toe_link"/>
-  <xacro:gen_toe name="front_right_toe_link"/>
-  <xacro:gen_toe name="rear_left_toe_link"/>
-  <xacro:gen_toe name="rear_right_toe_link"/>
-  <!-- Joints -->
-  <joint name="base_rear" type="fixed">
-    <parent link="base_link"/>
-    <child link="rear_link"/>
-  </joint>
   <joint name="base_front" type="fixed">
     <parent link="base_link"/>
     <child link="front_link"/>
   </joint>
-  <!-- Shoulder Joints -->
-  <xacro:gen_shoulder_joint pos="front_left" shiftx="-0.093" shifty="-0.036"/>
-  <xacro:gen_shoulder_joint pos="front_right" shiftx="-0.093" shifty="0.036"/>
-  <xacro:gen_shoulder_joint pos="rear_left" shiftx="0.093" shifty="-0.036"/>
-  <xacro:gen_shoulder_joint pos="rear_right" shiftx="0.093" shifty="0.036"/>
-  <!-- Leg Joints -->
-  <xacro:gen_leg_joint pos="front_left" shift="-0.042"/>
-  <xacro:gen_leg_joint pos="front_right" shift="0.042"/>
-  <xacro:gen_leg_joint pos="rear_left" shift="-0.042"/>
-  <xacro:gen_leg_joint pos="rear_right" shift="0.042"/>
-  <!-- Foot Joints -->
-  <xacro:gen_foot_joint pos="front_left"/>
-  <xacro:gen_foot_joint pos="front_right"/>
-  <xacro:gen_foot_joint pos="rear_left"/>
-  <xacro:gen_foot_joint pos="rear_right"/>
-  <!-- Toe Joints -->
-  <xacro:gen_toe_joint pos="front_left"/>
-  <xacro:gen_toe_joint pos="front_right"/>
-  <xacro:gen_toe_joint pos="rear_left"/>
-  <xacro:gen_toe_joint pos="rear_right"/>
+  <!-- create Legs -->
+  <xacro:gen_full_leg_joint pos="front_left" shiftx="-0.093" shifty="-0.036" shift="-0.042"/>
+  <xacro:gen_full_leg_joint pos="front_right" shiftx="-0.093" shifty="0.036" shift="0.042"/>
+  <xacro:gen_full_leg_joint pos="rear_left" shiftx="0.093" shifty="-0.036" shift="-0.042"/>
+  <xacro:gen_full_leg_joint pos="rear_right" shiftx="0.093" shifty="0.036" shift="0.042"/>
 </robot>

Commit message: added mass and dynamics

File: urdf/spotmicroai.urdf.xacro (robot description, xacro)
@@ -18,4 +18,9 @@
   <xacro:property name="shoulder_length" value="0.044" />
   <xacro:property name="shoulder_width" value="0.038" />
+  <xacro:property name="leg_length" value="0.120" />
+  <xacro:property name="foot_length" value="0.155" />
+  <xacro:property name="toe_radius" value="0.020" />
+  <!--  <xacro:property name="toe_radius" value="0.014" /> -->
+  <xacro:property name="toe_width" value="0.020" />
   <!-- Macros -->
   <xacro:macro name="gen_shoulder" params="name">
@@ -28,4 +33,14 @@
         <material name="black"/>
       </visual>
+      <collision>
+        <geometry>
+          <box size="${shoulder_length} ${shoulder_width} ${body_height}"/>
+        </geometry>
+        <origin rpy="0 0 0" xyz="0 0 0"/>
+      </collision>
+      <inertial>
+        <mass value="0.10"/>
+        <inertia ixx="100" ixy="0" ixz="0" iyy="100" iyz="0" izz="100" />
+      </inertial>
     </link>
   </xacro:macro>
@@ -34,9 +49,19 @@
       <visual>
         <geometry>
-          <box size="0.028 0.036 0.120"/>
-        </geometry>
-        <origin rpy="0 0 0" xyz="0 0 -0.050"/>
+          <box size="0.028 0.036 ${leg_length}"/>
+        </geometry>
+        <origin rpy="0.0 0.0 0.0" xyz="0.0 0.0 -0.050"/>
         <material name="yellow"/>
       </visual>
+      <collision>
+        <origin rpy="0.0 0.0 0.0" xyz="0.0 0.0 -0.050"/>
+        <geometry>
+          <box size="0.028 0.036 ${leg_length}"/>
+        </geometry>
+      </collision>
+      <inertial>
+        <mass value="0.10"/>
+        <inertia ixx="100" ixy="0" ixz="0" iyy="100" iyz="0" izz="100" />
+      </inertial>
     </link>
   </xacro:macro>
@@ -45,9 +70,19 @@
       <visual>
         <geometry>
-          <box size="0.026 0.020 0.155"/>
-        </geometry>
-        <origin rpy="0 0 0" xyz="0 0 -0.070"/>
+          <box size="0.026 0.020 ${foot_length}"/>
+        </geometry>
+        <origin rpy="0.0 0.0 0.0" xyz="0.0 0.0 -0.070"/>
         <material name="black"/>
       </visual>
+      <collision>
+        <geometry>
+          <box size="0.026 0.020 ${foot_length}"/>
+        </geometry>
+        <origin rpy="0.0 0.0 0.0" xyz="0.0 0.0 -0.070"/>
+      </collision>
+      <inertial>
+        <mass value="0.10"/>
+        <inertia ixx="100" ixy="0" ixz="0" iyy="100" iyz="0" izz="100" />
+      </inertial>
     </link>
   </xacro:macro>
@@ -56,9 +91,19 @@
       <visual>
         <geometry>
-          <cylinder length="0.020" radius="0.014"/>
+          <sphere radius="${toe_radius}" />
         </geometry>
         <origin rpy="1.5708 0 0" xyz="0 0 0"/>
         <material name="grey"/>
       </visual>
+      <collision>
+        <geometry>
+          <sphere radius="${toe_radius}" />
+        </geometry>
+        <origin rpy="1.5708 0 0" xyz="0 0 0"/>
+      </collision>
+      <inertial>
+        <mass value="0.01"/>
+        <inertia ixx="100" ixy="0" ixz="0" iyy="100" iyz="0" izz="100" />
+      </inertial>
     </link>
   </xacro:macro>
@@ -68,6 +113,7 @@
       <child link="${pos}_foot_link"/>
       <axis xyz="0 1 0"/>
-      <origin xyz="-0.01 0 -0.120"/>
+      <origin xyz="-0.01 0 -${leg_length}"/>
       <limit effort="1000.0" lower="-0.1" upper="2.59" velocity="0.5"/>
+      <dynamics damping="0.0" friction="0.0"/>
     </joint>
   </xacro:macro>
@@ -76,5 +122,5 @@
       <parent link="${pos}_foot_link"/>
       <child link="${pos}_toe_link"/>
-      <origin xyz="0 0 -0.155"/>
+      <origin xyz="0 0 -${foot_length}"/>
     </joint>
   </xacro:macro>
@@ -86,4 +132,5 @@
       <origin xyz="0 ${shift} 0"/>
       <limit effort="1000.0" lower="-2.666" upper="1.548" velocity="0.5"/>
+      <dynamics damping="0.0" friction="0.0"/>
     </joint>
   </xacro:macro>
@@ -95,4 +142,5 @@
       <origin xyz="${shiftx} ${shifty} 0"/>
       <limit effort="1000.0" lower="-0.548" upper="0.548" velocity="0.5"/>
+      <dynamics damping="0.0" friction="0.0"/>
     </joint>
   </xacro:macro>
@@ -116,4 +164,13 @@
       <origin rpy="0 0 0" xyz="0 0 0"/>
     </visual>
+    <collision>
+      <geometry>
+        <box size="${body_length} ${body_width} ${body_height}"/>
+      </geometry>
+    </collision>
+    <inertial>
+      <mass value="0.80"/>
+      <inertia ixx="100" ixy="0" ixz="0" iyy="100" iyz="0" izz="100" />
+    </inertial>
   </link>
   <link name="rear_link">
@@ -125,4 +182,14 @@
       <material name="yellow"/>
     </visual>
+    <collision>
+      <geometry>
+        <box size="${rear_length} ${body_width} ${body_height}"/>
+      </geometry>
+      <origin rpy="0 0 0" xyz="0.145 0 0"/>
+    </collision>
+    <inertial>
+      <mass value="0.20"/>
+      <inertia ixx="100" ixy="0" ixz="0" iyy="100" iyz="0" izz="100" />
+    </inertial>
   </link>
   <joint name="base_rear" type="fixed">
@@ -138,4 +205,14 @@
       <material name="yellow"/>
     </visual>
+    <collision>
+      <geometry>
+        <box size="${front_length} ${body_width} ${body_height}"/>
+      </geometry>
+      <origin rpy="0 0 0" xyz="-0.145 0 0"/>
+    </collision>
+    <inertial>
+      <mass value="0.20"/>
+      <inertia ixx="100" ixy="0" ixz="0" iyy="100" iyz="0" izz="100" />
+    </inertial>
   </link>
   <joint name="base_front" type="fixed">
