Commit message: URDF improvements

File: urdf/spotmicroai.urdf.xacro (robot description, xacro)
@@ -23,4 +23,7 @@
   <!--  <xacro:property name="toe_radius" value="0.014" /> -->
   <xacro:property name="toe_width" value="0.020" />
+  <xacro:property name="shift" value="0.052" />
+  <xacro:property name="shiftx" value="0.093" />
+  <xacro:property name="shifty" value="0.036" />
   <!-- Macros -->
   <xacro:macro name="gen_shoulder" params="name">
@@ -45,4 +48,14 @@
     </link>
   </xacro:macro>
+  <xacro:macro name="gen_shoulder_joint" params="pos shiftx shifty">
+    <joint name="${pos}_shoulder" type="revolute">
+      <parent link="base_link"/>
+      <child link="${pos}_shoulder_link"/>
+      <axis xyz="1 0 0"/>
+      <origin xyz="${shiftx} ${shifty} 0"/>
+      <limit effort="10000.0" lower="-0.548" upper="0.548" velocity="0.5"/>
+      <dynamics damping="0.0" friction="0.5"/>
+    </joint>
+  </xacro:macro>
   <xacro:macro name="gen_leg" params="name">
     <link name="${name}">
@@ -62,66 +75,7 @@
       <inertial>
         <mass value="0.10"/>
-        <inertia ixx="100" ixy="0" ixz="0" iyy="100" iyz="0" izz="100" />
-      </inertial>
-    </link>
-  </xacro:macro>
-  <xacro:macro name="gen_foot" params="name">
-    <link name="${name}">
-      <visual>
-        <geometry>
-          <box size="0.026 0.020 ${foot_length}"/>
-        </geometry>
-        <origin rpy="0.0 0.0 0.0" xyz="0.0 0.0 -0.070"/>
-        <material name="black"/>
-      </visual>
-      <collision>
-        <geometry>
-          <box size="0.026 0.020 ${foot_length}"/>
-        </geometry>
-        <origin rpy="0.0 0.0 0.0" xyz="0.0 0.0 -0.070"/>
-      </collision>
-      <inertial>
-        <mass value="0.10"/>
-        <inertia ixx="100" ixy="0" ixz="0" iyy="100" iyz="0" izz="100" />
-      </inertial>
-    </link>
-  </xacro:macro>
-  <xacro:macro name="gen_toe" params="name">
-    <link name="${name}">
-      <visual>
-        <geometry>
-          <sphere radius="${toe_radius}" />
-        </geometry>
-        <origin rpy="1.5708 0 0" xyz="0 0 0"/>
-        <material name="grey"/>
-      </visual>
-      <collision>
-        <geometry>
-          <sphere radius="${toe_radius}" />
-        </geometry>
-        <origin rpy="1.5708 0 0" xyz="0 0 0"/>
-      </collision>
-      <inertial>
-        <mass value="0.01"/>
-        <inertia ixx="100" ixy="0" ixz="0" iyy="100" iyz="0" izz="100" />
-      </inertial>
-    </link>
-  </xacro:macro>
-  <xacro:macro name="gen_foot_joint" params="pos">
-    <joint name="${pos}_foot" type="revolute">
-      <parent link="${pos}_leg_link"/>
-      <child link="${pos}_foot_link"/>
-      <axis xyz="0 1 0"/>
-      <origin xyz="-0.01 0 -${leg_length}"/>
-      <limit effort="1000.0" lower="-0.1" upper="2.59" velocity="0.5"/>
-      <dynamics damping="0.0" friction="0.0"/>
-    </joint>
-  </xacro:macro>
-  <xacro:macro name="gen_toe_joint" params="pos">
-    <joint name="${pos}_toe" type="fixed">
-      <parent link="${pos}_foot_link"/>
-      <child link="${pos}_toe_link"/>
-      <origin xyz="0 0 -${foot_length}"/>
-    </joint>
+        <inertia ixx="10" ixy="0" ixz="0" iyy="10" iyz="0" izz="10" />
+      </inertial>
+    </link>
   </xacro:macro>
   <xacro:macro name="gen_leg_joint" params="pos shift">
@@ -132,15 +86,64 @@
       <origin xyz="0 ${shift} 0"/>
       <limit effort="1000.0" lower="-2.666" upper="1.548" velocity="0.5"/>
+      <dynamics damping="0.0" friction="0.5"/>
+    </joint>
+  </xacro:macro>
+  <xacro:macro name="gen_foot" params="name">
+    <link name="${name}">
+      <visual>
+        <geometry>
+          <box size="0.026 0.020 ${foot_length}"/>
+        </geometry>
+        <origin rpy="0.0 0.0 0.0" xyz="0.0 0.0 -0.090"/>
+        <material name="black"/>
+      </visual>
+      <collision>
+        <geometry>
+          <box size="0.026 0.020 ${foot_length}"/>
+        </geometry>
+        <origin rpy="0.0 0.0 0.0" xyz="0.0 0.0 -0.090"/>
+      </collision>
+      <inertial>
+        <mass value="0.15"/>
+        <inertia ixx="1" ixy="0" ixz="0" iyy="1" iyz="0" izz="1" />
+      </inertial>
+    </link>
+  </xacro:macro>
+  <xacro:macro name="gen_foot_joint" params="pos">
+    <joint name="${pos}_foot" type="revolute">
+      <parent link="${pos}_leg_link"/>
+      <child link="${pos}_foot_link"/>
+      <axis xyz="0 1 0"/>
+      <origin xyz="-0.01 0 -${leg_length+0.20}"/>
+      <limit effort="1000.0" lower="-0.1" upper="2.59" velocity="0.5"/>
       <dynamics damping="0.0" friction="0.0"/>
     </joint>
   </xacro:macro>
-  <xacro:macro name="gen_shoulder_joint" params="pos shiftx shifty">
-    <joint name="${pos}_shoulder" type="revolute">
-      <parent link="base_link"/>
-      <child link="${pos}_shoulder_link"/>
-      <axis xyz="1 0 0"/>
-      <origin xyz="${shiftx} ${shifty} 0"/>
-      <limit effort="1000.0" lower="-0.548" upper="0.548" velocity="0.5"/>
-      <dynamics damping="0.0" friction="0.0"/>
+  <xacro:macro name="gen_toe" params="name">
+    <link name="${name}">
+      <visual>
+        <geometry>
+          <sphere radius="${toe_radius}" />
+        </geometry>
+        <origin rpy="1.5708 0 0" xyz="0 0 0"/>
+        <material name="grey"/>
+      </visual>
+      <collision>
+        <geometry>
+          <sphere radius="${toe_radius}" />
+        </geometry>
+        <origin rpy="1.5708 0 0" xyz="0 0 0"/>
+      </collision>
+      <inertial>
+        <mass value="0.01"/>
+        <inertia ixx="100" ixy="0" ixz="0" iyy="100" iyz="0" izz="100" />
+      </inertial>
+    </link>
+  </xacro:macro>
+ <xacro:macro name="gen_toe_joint" params="pos">
+    <joint name="${pos}_toe" type="fixed">
+      <parent link="${pos}_foot_link"/>
+      <child link="${pos}_toe_link"/>
+      <origin xyz="0 0 -${foot_length}"/>
     </joint>
   </xacro:macro>
@@ -221,7 +224,7 @@
   </joint>
   <!-- create Legs -->
-  <xacro:gen_full_leg_joint pos="front_left" shiftx="-0.093" shifty="-0.036" shift="-0.042"/>
-  <xacro:gen_full_leg_joint pos="front_right" shiftx="-0.093" shifty="0.036" shift="0.042"/>
-  <xacro:gen_full_leg_joint pos="rear_left" shiftx="0.093" shifty="-0.036" shift="-0.042"/>
-  <xacro:gen_full_leg_joint pos="rear_right" shiftx="0.093" shifty="0.036" shift="0.042"/>
+  <xacro:gen_full_leg_joint pos="front_left" shiftx="-${shiftx}" shifty="-${shifty}" shift="-${shift}"/>
+  <xacro:gen_full_leg_joint pos="front_right" shiftx="-${shiftx}" shifty="${shifty}" shift="${shift}"/>
+  <xacro:gen_full_leg_joint pos="rear_left" shiftx="${shiftx}" shifty="-${shifty}" shift="-${shift}"/>
+  <xacro:gen_full_leg_joint pos="rear_right" shiftx="${shiftx}" shifty="${shifty}" shift="${shift}"/>
 </robot>

Commit message: Playing with dynamics

File: urdf/spotmicroai.urdf.xacro (robot description, xacro)
@@ -54,5 +54,5 @@
       <axis xyz="1 0 0"/>
       <origin xyz="${shiftx} ${shifty} 0"/>
-      <limit effort="10000.0" lower="-0.548" upper="0.548" velocity="0.5"/>
+      <limit effort="1000.0" lower="-0.548" upper="0.548" velocity="0.7"/>
       <dynamics damping="0.0" friction="0.5"/>
     </joint>
@@ -74,6 +74,6 @@
       </collision>
       <inertial>
-        <mass value="0.10"/>
-        <inertia ixx="10" ixy="0" ixz="0" iyy="10" iyz="0" izz="10" />
+        <mass value="0.15"/>
+        <inertia ixx="1000" ixy="0" ixz="0" iyy="1000" iyz="0" izz="1000" />
       </inertial>
     </link>
@@ -86,5 +86,5 @@
       <origin xyz="0 ${shift} 0"/>
       <limit effort="1000.0" lower="-2.666" upper="1.548" velocity="0.5"/>
-      <dynamics damping="0.0" friction="0.5"/>
+      <dynamics damping="0.0" friction="0.0"/>
     </joint>
   </xacro:macro>
@@ -105,6 +105,6 @@
       </collision>
       <inertial>
-        <mass value="0.15"/>
-        <inertia ixx="1" ixy="0" ixz="0" iyy="1" iyz="0" izz="1" />
+        <mass value="0.1"/>
+        <inertia ixx="1000" ixy="0" ixz="0" iyy="1000" iyz="0" izz="1000" />
       </inertial>
     </link>
@@ -115,7 +115,7 @@
       <child link="${pos}_foot_link"/>
       <axis xyz="0 1 0"/>
-      <origin xyz="-0.01 0 -${leg_length+0.20}"/>
+      <origin xyz="-0.01 0 -${leg_length}"/>
       <limit effort="1000.0" lower="-0.1" upper="2.59" velocity="0.5"/>
-      <dynamics damping="0.0" friction="0.0"/>
+      <dynamics damping="0.0" friction="0.5"/>
     </joint>
   </xacro:macro>
@@ -137,5 +137,5 @@
       <inertial>
         <mass value="0.01"/>
-        <inertia ixx="100" ixy="0" ixz="0" iyy="100" iyz="0" izz="100" />
+        <inertia ixx="1000" ixy="0" ixz="0" iyy="1000" iyz="0" izz="1000" />
       </inertial>
     </link>
@@ -145,5 +145,5 @@
       <parent link="${pos}_foot_link"/>
       <child link="${pos}_toe_link"/>
-      <origin xyz="0 0 -${foot_length}"/>
+      <origin xyz="0 0 -${foot_length+0.01}"/>
     </joint>
   </xacro:macro>

Commit message: Simulation

File: urdf/spotmicroai.urdf.xacro (robot description, xacro)
@@ -53,5 +53,5 @@
       <child link="${pos}_shoulder_link"/>
       <axis xyz="1 0 0"/>
-      <origin xyz="${shiftx} ${shifty} 0"/>
+      <origin rpy="0 0 0" xyz="${shiftx} ${shifty} 0"/>
       <limit effort="1000.0" lower="-0.548" upper="0.548" velocity="0.7"/>
       <dynamics damping="0.0" friction="0.5"/>
@@ -84,5 +84,5 @@
       <child link="${pos}_leg_link"/>
       <axis xyz="0 1 0"/>
-      <origin xyz="0 ${shift} 0"/>
+      <origin rpy="0 0 0" xyz="0 ${shift} 0"/>
       <limit effort="1000.0" lower="-2.666" upper="1.548" velocity="0.5"/>
       <dynamics damping="0.0" friction="0.0"/>
@@ -115,5 +115,5 @@
       <child link="${pos}_foot_link"/>
       <axis xyz="0 1 0"/>
-      <origin xyz="-0.01 0 -${leg_length}"/>
+      <origin rpy="0 0 0" xyz="-0.01 0 -${leg_length}"/>
       <limit effort="1000.0" lower="-0.1" upper="2.59" velocity="0.5"/>
       <dynamics damping="0.0" friction="0.5"/>
@@ -134,4 +134,5 @@
         </geometry>
         <origin rpy="1.5708 0 0" xyz="0 0 0"/>
+        <contact_coefficients mu="10"/>
       </collision>
       <inertial>

Commit message: Code cleanups

File: urdf/spotmicroai.urdf.xacro (robot description, xacro)
@@ -134,8 +134,8 @@
         </geometry>
         <origin rpy="1.5708 0 0" xyz="0 0 0"/>
-        <contact_coefficients mu="10"/>
-      </collision>
-      <inertial>
-        <mass value="0.01"/>
+        <contact_coefficients mu="0.8" />
+      </collision>
+      <inertial>
+        <mass value="0.05"/>
         <inertia ixx="1000" ixy="0" ixz="0" iyy="1000" iyz="0" izz="1000" />
       </inertial>

Commit message: STL

File: urdf/spotmicroai.urdf.xacro (robot description, xacro)
@@ -15,5 +15,5 @@
   <xacro:property name="body_height" value="0.070" />
   <xacro:property name="front_length" value="0.058" />
-  <xacro:property name="rear_length" value="0.057" />
+  <xacro:property name="rear_length" value="0.040" />
   <xacro:property name="shoulder_length" value="0.044" />
   <xacro:property name="shoulder_width" value="0.038" />
@@ -181,7 +181,8 @@
     <visual>
       <geometry>
-        <box size="${rear_length} ${body_width} ${body_height}"/>
-      </geometry>
-      <origin rpy="0 0 0" xyz="0.145 0 0"/>
+              <mesh filename="../STL/files/R_cover.stl" scale="0.001 0.001 0.001"/>
+        <!--<box size="${rear_length} ${body_width} ${body_height}"/> -->
+      </geometry>
+      <origin rpy="0 0 0" xyz="0.120 0 0"/>
       <material name="yellow"/>
     </visual>
@@ -190,5 +191,5 @@
         <box size="${rear_length} ${body_width} ${body_height}"/>
       </geometry>
-      <origin rpy="0 0 0" xyz="0.145 0 0"/>
+      <origin rpy="0 0 0" xyz="0.135 0 0"/>
     </collision>
     <inertial>
@@ -204,7 +205,8 @@
     <visual>
       <geometry>
-        <box size="${front_length} ${body_width} ${body_height}"/>
-      </geometry>
-      <origin rpy="0 0 0" xyz="-0.145 0 0"/>
+        <mesh filename="../STL/files/F_cover.stl" scale="0.001 0.001 0.001"/>
+<!--        <box size="${front_length} ${body_width} ${body_height}"/> -->
+      </geometry>
+      <origin rpy="0 0 0" xyz="-0.130 0 0"/>
       <material name="yellow"/>
     </visual>

Commit message: Lidar added to URDF

File: urdf/spotmicroai.urdf.xacro (robot description, xacro)
@@ -14,4 +14,7 @@
   <xacro:property name="body_width" value="0.110" />
   <xacro:property name="body_height" value="0.070" />
+  <xacro:property name="lidar_length" value="0.0985" />
+  <xacro:property name="lidar_width" value="0.0577" />
+  <xacro:property name="lidar_height" value="0.070" />
   <xacro:property name="front_length" value="0.058" />
   <xacro:property name="rear_length" value="0.040" />
@@ -178,4 +181,28 @@
     </inertial>
   </link>
+  <!-- Lidar Backpack -->
+   <link name="lidar_link">
+    <visual>
+      <geometry>
+        <mesh filename="../STL/lidar/rplidar_main.STL" scale="0.001 0.001 0.001"/>
+      </geometry>
+      <material name="black"/>
+      <origin rpy="1.57075 0 0" xyz="${-lidar_length/2-0.015} ${lidar_width/2} ${body_height/2}"/>
+    </visual>
+    <collision>
+      <geometry>
+        <box size="${lidar_length} ${lidar_width} ${lidar_height}"/>
+      </geometry>
+      <origin rpy="0 0 0" xyz="0 0 ${body_height/2}"/>
+    </collision>
+    <inertial>
+      <mass value="0.50"/>
+      <inertia ixx="100" ixy="0" ixz="0" iyy="100" iyz="0" izz="100" />
+    </inertial>
+  </link>
+  <joint name="base_lidar" type="fixed">
+    <parent link="base_link"/>
+    <child link="lidar_link"/>
+  </joint>
   <link name="rear_link">
     <visual>

Commit message: Jetson Nano Code

File: urdf/spotmicroai.urdf.xacro (robot description, xacro)
@@ -30,5 +30,5 @@
   <xacro:property name="shifty" value="0.036" />
   <!-- Macros -->
-  <xacro:macro name="gen_shoulder" params="name">
+  <xacro:macro name="gen_shoulder" params="name left">
     <link name="${name}">
       <visual>
@@ -36,4 +36,19 @@
           <box size="${shoulder_length} ${shoulder_width} ${body_height}"/>
         </geometry>
+        <origin rpy="0 0 0" xyz="0 0 0"/>
+<!--
+        <xacro:if value="${left}">
+        <geometry>
+          <mesh filename="../STL/files/L_arm_joint.stl" scale="0.001 0.001 0.001"/>
+        </geometry>
+        <origin rpy="0 0 -1.57075" xyz="0 0.01 -0.02"/>
+        </xacro:if>
+        <xacro:unless value="${left}">
+        <geometry>
+          <mesh filename="../STL/files/R_arm_joint.stl" scale="0.001 0.001 0.001"/>
+        </geometry>
+        <origin rpy="0 0 -1.57075" xyz="0 0 0"/>
+        </xacro:unless>
+        -->
         <origin rpy="0 0 0" xyz="0 0 0"/>
         <material name="black"/>
@@ -127,14 +142,14 @@
       <visual>
         <geometry>
+        <mesh filename="../STL/files/foot.stl" scale="0.001 0.001 0.001"/>
+        </geometry>
+        <origin rpy="0 0 0" xyz="0 -0.01 0"/>
+        <material name="grey"/>
+      </visual>
+      <collision>
+        <geometry>
           <sphere radius="${toe_radius}" />
         </geometry>
-        <origin rpy="1.5708 0 0" xyz="0 0 0"/>
-        <material name="grey"/>
-      </visual>
-      <collision>
-        <geometry>
-          <sphere radius="${toe_radius}" />
-        </geometry>
-        <origin rpy="1.5708 0 0" xyz="0 0 0"/>
+        <origin rpy="0 0 0" xyz="0 0 0"/>
         <contact_coefficients mu="0.8" />
       </collision>
@@ -152,6 +167,6 @@
     </joint>
   </xacro:macro>
-  <xacro:macro name="gen_full_leg_joint" params="pos shiftx shifty shift">
-    <xacro:gen_shoulder name="${pos}_shoulder_link"/>
+  <xacro:macro name="gen_full_leg_joint" params="pos shiftx shifty shift left">
+    <xacro:gen_shoulder name="${pos}_shoulder_link" left="${left}"/>
     <xacro:gen_leg name="${pos}_leg_link"/>
     <xacro:gen_foot name="${pos}_foot_link"/>
@@ -254,7 +269,7 @@
   </joint>
   <!-- create Legs -->
-  <xacro:gen_full_leg_joint pos="front_left" shiftx="-${shiftx}" shifty="-${shifty}" shift="-${shift}"/>
-  <xacro:gen_full_leg_joint pos="front_right" shiftx="-${shiftx}" shifty="${shifty}" shift="${shift}"/>
-  <xacro:gen_full_leg_joint pos="rear_left" shiftx="${shiftx}" shifty="-${shifty}" shift="-${shift}"/>
-  <xacro:gen_full_leg_joint pos="rear_right" shiftx="${shiftx}" shifty="${shifty}" shift="${shift}"/>
+  <xacro:gen_full_leg_joint pos="front_left" shiftx="-${shiftx}" shifty="-${shifty}" shift="-${shift}" left="true"/>
+  <xacro:gen_full_leg_joint pos="front_right" shiftx="-${shiftx}" shifty="${shifty}" shift="${shift}" left="false"/>
+  <xacro:gen_full_leg_joint pos="rear_left" shiftx="${shiftx}" shifty="-${shifty}" shift="-${shift}" left="true"/>
+  <xacro:gen_full_leg_joint pos="rear_right" shiftx="${shiftx}" shifty="${shifty}" shift="${shift}" left="false"/>
 </robot>

Commit message: trotting gait

File: urdf/spotmicroai.urdf.xacro (robot description, xacro)
@@ -203,5 +203,5 @@
       </geometry>
       <material name="black"/>
-      <origin rpy="1.57075 0 0" xyz="${-lidar_length/2-0.015} ${lidar_width/2} ${body_height/2}"/>
+      <origin rpy="1.57075 0 0" xyz="${-lidar_length/2-0.015} ${lidar_width/2} 0"/>
     </visual>
     <collision>
@@ -209,5 +209,5 @@
         <box size="${lidar_length} ${lidar_width} ${lidar_height}"/>
       </geometry>
-      <origin rpy="0 0 0" xyz="0 0 ${body_height/2}"/>
+      <origin rpy="0 0 0" xyz="0 0 0"/>
     </collision>
     <inertial>
@@ -219,4 +219,5 @@
     <parent link="base_link"/>
     <child link="lidar_link"/>
+        <origin xyz="0 0 ${body_height/2}"/>
   </joint>
   <link name="rear_link">

Commit message: using the real model - almost finished

File: urdf/spotmicroai.urdf.xacro (robot description, xacro)
@@ -22,5 +22,5 @@
   <xacro:property name="shoulder_width" value="0.038" />
   <xacro:property name="leg_length" value="0.120" />
-  <xacro:property name="foot_length" value="0.155" />
+  <xacro:property name="foot_length" value="0.105" />
   <xacro:property name="toe_radius" value="0.020" />
   <!--  <xacro:property name="toe_radius" value="0.014" /> -->
@@ -33,23 +33,16 @@
     <link name="${name}">
       <visual>
-        <geometry>
-          <box size="${shoulder_length} ${shoulder_width} ${body_height}"/>
-        </geometry>
-        <origin rpy="0 0 0" xyz="0 0 0"/>
-<!--
         <xacro:if value="${left}">
         <geometry>
-          <mesh filename="../STL/files/L_arm_joint.stl" scale="0.001 0.001 0.001"/>
-        </geometry>
-        <origin rpy="0 0 -1.57075" xyz="0 0.01 -0.02"/>
+          <mesh filename="../Parts/lshoulder.stl" scale="0.001 0.001 0.001"/>
+        </geometry>
+        <origin rpy="0 0 0" xyz="-0.135 -0.02 -0.01"/>
         </xacro:if>
         <xacro:unless value="${left}">
         <geometry>
-          <mesh filename="../STL/files/R_arm_joint.stl" scale="0.001 0.001 0.001"/>
-        </geometry>
-        <origin rpy="0 0 -1.57075" xyz="0 0 0"/>
+          <mesh filename="../Parts/rshoulder.stl" scale="0.001 0.001 0.001"/>
+        </geometry>
+        <origin rpy="0 0 0" xyz="-0.135 -0.09 -0.01"/>
         </xacro:unless>
-        -->
-        <origin rpy="0 0 0" xyz="0 0 0"/>
         <material name="black"/>
       </visual>
@@ -110,8 +103,16 @@
     <link name="${name}">
       <visual>
-        <geometry>
-          <box size="0.026 0.020 ${foot_length}"/>
-        </geometry>
-        <origin rpy="0.0 0.0 0.0" xyz="0.0 0.0 -0.090"/>
+        <xacro:if value="${left}">
+        <geometry>
+          <mesh filename="../Parts/lfoot.stl" scale="0.001 0.001 0.001"/>
+        </geometry>
+        <origin rpy="0 0 0" xyz="-0.120 0.04 0.1"/>
+        </xacro:if>
+        <xacro:unless value="${left}">
+        <geometry>
+          <mesh filename="../Parts/rfoot.stl" scale="0.001 0.001 0.001"/>
+        </geometry>
+        <origin rpy="0 0 0" xyz="-0.120 -0.15 0.1"/>
+        </xacro:unless>
         <material name="black"/>
       </visual>
@@ -144,5 +145,5 @@
         <mesh filename="../STL/files/foot.stl" scale="0.001 0.001 0.001"/>
         </geometry>
-        <origin rpy="0 0 0" xyz="0 -0.01 0"/>
+        <origin rpy="0 -0.40010 0" xyz="0 -0.01 0"/>
         <material name="grey"/>
       </visual>
@@ -181,16 +182,17 @@
     <visual>
       <geometry>
+        <mesh filename="../Parts/mainbody.stl" scale="0.001 0.001 0.001"/>
+      </geometry>
+      <material name="black"/>
+      <origin rpy="0 0 0" xyz="-0.045 -0.060 -0.015"/>
+    </visual>
+    <collision>
+      <geometry>
         <box size="${body_length} ${body_width} ${body_height}"/>
       </geometry>
-      <material name="yellow"/>
       <origin rpy="0 0 0" xyz="0 0 0"/>
-    </visual>
-    <collision>
-      <geometry>
-        <box size="${body_length} ${body_width} ${body_height}"/>
-      </geometry>
-    </collision>
-    <inertial>
-      <mass value="0.80"/>
+    </collision>
+    <inertial>
+      <mass value="2.80"/>
       <inertia ixx="100" ixy="0" ixz="0" iyy="100" iyz="0" izz="100" />
     </inertial>
@@ -224,8 +226,7 @@
     <visual>
       <geometry>
-              <mesh filename="../STL/files/R_cover.stl" scale="0.001 0.001 0.001"/>
-        <!--<box size="${rear_length} ${body_width} ${body_height}"/> -->
-      </geometry>
-      <origin rpy="0 0 0" xyz="0.120 0 0"/>
+        <mesh filename="../Parts/backpart.stl" scale="0.001 0.001 0.001"/>
+      </geometry>
+      <origin rpy="0 0 0" xyz="-0.040 -0.060 -0.0140"/>
       <material name="yellow"/>
     </visual>
@@ -248,8 +249,7 @@
     <visual>
       <geometry>
-        <mesh filename="../STL/files/F_cover.stl" scale="0.001 0.001 0.001"/>
-<!--        <box size="${front_length} ${body_width} ${body_height}"/> -->
-      </geometry>
-      <origin rpy="0 0 0" xyz="-0.130 0 0"/>
+        <mesh filename="../Parts/frontpart.stl" scale="0.001 0.001 0.001"/>
+      </geometry>
+      <origin rpy="0 0 0" xyz="-0.040 -0.060 -0.0140"/>
       <material name="yellow"/>
     </visual>
